File: Load-emulator/v1.1/currentSink1A.kicad_sch (KiCad schematic)
At the start: 3 parts, among them Q2 TIP41C, U14 LM318H

Commit message: Todos erros foram consertados, assim como todos os avisos, com exceção dos que se referem ao PC104, que teve seu footprint modificado. Todos modelos 3D foram corretamente upados. Adição de zonas de GND.
Parts:
- R18: footprint Resistor_SMD:R_0201_0603Metric -> Resistor_THT:R_Axial_DIN0207_L6.3mm_D2.5mm_P2.54mm_Vertical
- U14: footprint LM318M:SOIC127P599X175-8N -> footprints:SOIC127P599X175-8N
Changed lines of the file:
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@@
 			)
 		)
-		(property "Footprint" "LM318M:SOIC127P599X175-8N"
+		(property "Footprint" "footprints:SOIC127P599X175-8N"
 			(at 135.89 85.09 0)
 			(effects
@@
 			)
 		)
-		(property "Footprint" "Resistor_SMD:R_0201_0603Metric"
+		(property "Footprint" "Resistor_THT:R_Axial_DIN0207_L6.3mm_D2.5mm_P2.54mm_Vertical"
 			(at 163.576 101.854 90)
 			(effects
