File: Load-emulator/v2.0/Filter_and_CurrentSink_2x1A.kicad_sch (KiCad schematic)
At the start: 18 parts, among them Q5 RD3L08DBLHRB, Q7 RD3L08DBLHRB, U10 INA185, U11 INA185, U7 LT1492, U8 LT1492

Commit message: [v2.0 - WIP] Added PCB Sketch
[REMOVED]
 - Some comments;

[ADDED]
- 3D models for some components, like heatsinks;
- PCB Sketch (This is just to review how it will look);
Parts:
- R18, R19, R20, R21: footprint (none) -> Resistor_SMD:R_0603_1608Metric
- U7, U8: footprint (none) -> footprints:SO-8_S_LIT
Changed lines of the file:
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@@
 	(title_block
 		(title "Load Emulator")
-		(date "2025-09-28")
+		(date "2025-10-03")
 		(rev "v2.0 - WIP")
 		(company "Spacelab")
@@
 		(polyline
 			(pts
-				(xy 121.285 20.32) (xy 203.835 20.32) (xy 203.835 121.92) (xy 121.285 121.92)
+				(xy 12.7 130.81) (xy 12.7 102.87) (xy 57.15 102.87) (xy 57.15 130.81)
 			)
 			(stroke
@@
 		(polyline
 			(pts
-				(xy 12.7 130.81) (xy 12.7 102.87) (xy 57.15 102.87) (xy 57.15 130.81)
+				(xy 58.42 165.4175) (xy 133.35 165.4174) (xy 133.35 197.8024) (xy 58.42 197.8025)
 			)
 			(stroke
@@
 		(polyline
 			(pts
-				(xy 12.7 165.4174) (xy 57.15 165.4174) (xy 57.15 197.8024) (xy 12.7 197.8024)
+				(xy 95.885 20.32) (xy 95.885 63.5) (xy 20.955 63.5) (xy 20.955 20.32)
 			)
 			(stroke
@@
 		(polyline
 			(pts
-				(xy 12.7 132.3975) (xy 57.15 132.3975) (xy 57.15 164.7825) (xy 12.7 164.7825)
+				(xy 121.285 20.32) (xy 203.835 20.32) (xy 203.835 121.92) (xy 121.285 121.92)
 			)
 			(stroke
@@
 		(polyline
 			(pts
-				(xy 221.615 45.72) (xy 268.605 45.72) (xy 268.605 129.54) (xy 221.615 129.54)
+				(xy 12.7 165.4174) (xy 57.15 165.4174) (xy 57.15 197.8024) (xy 12.7 197.8024)
 			)
 			(stroke
 				(width 0.25)
 				(type dash)
-				(color 255 0 0 1)
+				(color 0 0 0 1)
 			)
 			(fill
@@
 		(polyline
 			(pts
-				(xy 95.885 20.32) (xy 95.885 63.5) (xy 20.955 63.5) (xy 20.955 20.32)
+				(xy 12.7 132.3975) (xy 57.15 132.3975) (xy 57.15 164.7825) (xy 12.7 164.7825)
 			)
 			(stroke
@@
 		(polyline
 			(pts
-				(xy 58.42 165.4175) (xy 133.35 165.4174) (xy 133.35 197.8024) (xy 58.42 197.8025)
+				(xy 221.615 45.72) (xy 268.605 45.72) (xy 268.605 129.54) (xy 221.615 129.54)
 			)
 			(stroke
 				(width 0.25)
 				(type dash)
-				(color 0 0 0 1)
+				(color 255 0 0 1)
 			)
 			(fill
@@
 			)
 		)
-		(property "Footprint" ""
+		(property "Footprint" "footprints:SO-8_S_LIT"
 			(at 82.55 149.86 0)
 			(effects
@@
 			)
 		)
-		(property "Footprint" ""
+		(property "Footprint" "Resistor_SMD:R_0603_1608Metric"
 			(at 101.6 185.42 0)
 			(effects
@@
 			)
 		)
-		(property "Footprint" ""
+		(property "Footprint" "Resistor_SMD:R_0603_1608Metric"
 			(at 68.58 177.8 0)
 			(effects
@@
 			)
 		)
-		(property "Footprint" ""
+		(property "Footprint" "footprints:SO-8_S_LIT"
 			(at 68.58 149.86 0)
 			(effects
@@
 			)
 		)
-		(property "Footprint" ""
+		(property "Footprint" "Resistor_SMD:R_0603_1608Metric"
 			(at 101.6 177.8 0)
 			(effects
@@
 			)
 		)
-		(property "Footprint" ""
+		(property "Footprint" "footprints:SO-8_S_LIT"
 			(at 85.09 184.15 0)
 			(effects
@@
 			)
 		)
-		(property "Footprint" ""
+		(property "Footprint" "footprints:SO-8_S_LIT"
 			(at 157.48 40.64 0)
 			(effects
@@
 			)
 		)
-		(property "Footprint" ""
+		(property "Footprint" "footprints:SO-8_S_LIT"
 			(at 118.11 184.15 0)
 			(effects
@@
 			)
 		)
-		(property "Footprint" ""
+		(property "Footprint" "footprints:SO-8_S_LIT"
 			(at 157.48 82.55 0)
 			(effects
@@
 			)
 		)
-		(property "Footprint" ""
+		(property "Footprint" "Resistor_SMD:R_0603_1608Metric"
 			(at 68.58 185.42 0)
 			(effects

Commit message: [v2.0 - WIP] Release Candidate 1. (#6)
Ready for review
- PCB Wired up.
- Schematic ready.

[MISSING]
- Values for some Resistors and Capacitors;
- Verify if EPS conector is correct;
- Change schematic to release.
Parts:
- removed U10, U11: INA185, Package_TO_SOT_SMD:SOT-563, symbol Amplifier_Current:INA185
- C10: renamed from C33; footprint Capacitor_SMD:C_0201_0603Metric -> Capacitor_SMD:C_0805_2012Metric
- C11: renamed from C34; footprint Capacitor_SMD:C_0201_0603Metric -> Capacitor_SMD:C_0805_2012Metric
- HS4: renamed from HS6; footprint (none) -> footprints:573100D00000G
- HS5: footprint (none) -> footprints:573100D00000G
- R34: renamed from R56; footprint Resistor_SMD:R_0201_0603Metric -> Resistor_SMD:R_0603_1608Metric
- R35: renamed from R58; footprint Resistor_SMD:R_0201_0603Metric -> Resistor_SMD:R_0603_1608Metric
- R40: renamed from R60; footprint (none) -> Resistor_SMD:R_2512_6332Metric
- R41: renamed from R61; footprint (none) -> Resistor_SMD:R_2512_6332Metric
- renumbered Q5 to Q4, Q7 to Q5, R18 to R36, R19 to R37, R20 to R38, R21 to R39
Connections:
- no-connect marks 2 -> 0
Other:
- note added: "Resistor in Current Sink choose from: Rsense = (Vcontrol/Ieps)/10 Rsense = PWM/1A"
- note removed: "CURRENT SENSORs"
- note removed: "It's gonna be necessary to do alot to get the readings from the sensors, gonna need a ADC converter for the i²C, asked by Joao."
- note removed: "NOT ON PROTOTYPE"
- note removed: "Resistor in Current Sink choose from: Ieps = Vcontrol/Rsense Rsense = Vcontrol/Ieps Rsense = PWM/1A"
- moved on the sheet: Q4, Q5, R40, R41, U7A, U8A

Commit message: v2.0
Parts:
- C10, C11, R34, R35, R36, R37, R38, R39, R40, R41: Type (none) -> SMD
- HS4, HS5: Manufacturer (none) -> Boyd Laconia, LLC; Manufacturer Order Number (none) -> 573100D00000G; Type (none) -> SMD
- Q4, Q5: Manufacturer (none) -> Rohm Semiconductor; Manufacturer Order Number (none) -> RD3L08DBLHRBTL; Type (none) -> SMD
- U7, U8: Manufacturer (none) -> Analog Devices Inc.; Manufacturer Order Number (none) -> LT1492CS8#TRPBF; Type (none) -> SMD
